File: rocket2-trs.kicad_pcb (KiCad board)
At the start: 4 copper layers, 50 x 80 mm, 45 parts, among them J2 SMA, J3 ARM Cortex Debug, U4 AZ1117-3.3, Y1 16MHz

Commit message: Add LED
Parts:
- added D3: LED, Diode_SMD:D_0603_1608Metric, F.Cu at (227.3, 66.5)
- added R4: 1K, Resistor_SMD:R_0603_1608Metric, F.Cu at (224.3, 65.7)
Connections:
- U1 pad 45: unconnected-(U1-PB8-Pad45) -> Net-(U1-PB8)
Routing:
- net Net-(U1-PB8): track 0.00 -> 3.33 mm
- net Net-(D3-A): track 0.00 -> 2.18 mm
- net GND: vias 41 -> 42
Changed lines of the file:
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@@
   (net 44 "unconnected-(U1-PB6-Pad42)")
   (net 45 "unconnected-(U1-PB7-Pad43)")
-  (net 46 "unconnected-(U1-PB8-Pad45)")
+  (net 46 "Net-(D3-A)")
   (net 47 "unconnected-(U1-PB9-Pad46)")
   (net 48 "unconnected-(Y1-Pad1)")
+  (net 49 "Net-(U1-PB8)")
   (footprint "Capacitor_SMD:C_0603_1608Metric" (layer "F.Cu")
     (at 192 97.6 -90)
@@
       (net 2 "GND") (pinfunction "BOOT0") (pintype "input"))
     (pad "45" smd roundrect (at -1.25 -4.1625 270) (size 0.3 1.475) (layers "F.Cu" "F.Paste" "F.Mask") (roundrect_rratio 0.25)
-      (net 46 "unconnected-(U1-PB8-Pad45)") (pinfunction "PB8") (pintype "bidirectional+no_connect"))
+      (net 49 "Net-(U1-PB8)") (pinfunction "PB8") (pintype "bidirectional"))
     (pad "46" smd roundrect (at -1.75 -4.1625 270) (size 0.3 1.475) (layers "F.Cu" "F.Paste" "F.Mask") (roundrect_rratio 0.25)
       (net 47 "unconnected-(U1-PB9-Pad46)") (pinfunction "PB9") (pintype "bidirectional+no_connect"))
@@
       (net 2 "GND") (pintype "passive"))
     (model "${KICAD6_3DMODEL_DIR}/Capacitor_SMD.3dshapes/C_0603_1608Metric.wrl"
+      (offset (xyz 0 0 0))
+      (scale (xyz 1 1 1))
+      (rotate (xyz 0 0 0))
+    )
+  )
+  (footprint "Diode_SMD:D_0603_1608Metric" (layer "F.Cu")
+    (at 227.3 66.5 90)
+    (descr "Diode SMD 0603 (1608 Metric), square (rectangular) end terminal, IPC_7351 nominal, (Body size source: http://www.tortai-tech.com/upload/download/2011102023233369053.pdf), generated with kicad-footprint-generator")
+    (tags "diode")
+    (property "Manufacturer" "Generic")
+    (property "Part #" "Generic 0603 Red LED")
+    (property "Sheetfile" "rocket2-trs.kicad_sch")
+    (property "Sheetname" "")
+    (property "ki_description" "Light emitting diode, small symbol")
+    (property "ki_keywords" "LED diode light-emitting-diode")
+    (attr smd)
+    (fp_text reference "D3" (at 0 -1.43 90) (layer "F.SilkS") hide
+        (effects (font (size 1 1) (thickness 0.15)))
+    )
+    (fp_text value "LED" (at 0 1.43 90) (layer "F.Fab")
+        (effects (font (size 1 1) (thickness 0.15)))
+    )
+    (fp_text user "${REFERENCE}" (at 0 0 90) (layer "F.Fab")
+        (effects (font (size 0.4 0.4) (thickness 0.06)))
+    )
+    (fp_line (start -1.485 -0.735) (end -1.485 0.735)
+      (stroke (width 0.12) (type solid)) (layer "F.SilkS"))
+    (fp_line (start -1.485 0.735) (end 0.8 0.735)
+      (stroke (width 0.12) (type solid)) (layer "F.SilkS"))
+    (fp_line (start 0.8 -0.735) (end -1.485 -0.735)
+      (stroke (width 0.12) (type solid)) (layer "F.SilkS"))
+    (fp_line (start -1.48 -0.73) (end 1.48 -0.73)
+      (stroke (width 0.05) (type solid)) (layer "F.CrtYd"))
+    (fp_line (start -1.48 0.73) (end -1.48 -0.73)
+      (stroke (width 0.05) (type solid)) (layer "F.CrtYd"))
+    (fp_line (start 1.48 -0.73) (end 1.48 0.73)
+      (stroke (width 0.05) (type solid)) (layer "F.CrtYd"))
+    (fp_line (start 1.48 0.73) (end -1.48 0.73)
+      (stroke (width 0.05) (type solid)) (layer "F.CrtYd"))
+    (fp_line (start -0.8 -0.1) (end -0.8 0.4)
+      (stroke (width 0.1) (type solid)) (layer "F.Fab"))
+    (fp_line (start -0.8 0.4) (end 0.8 0.4)
+      (stroke (width 0.1) (type solid)) (layer "F.Fab"))
+    (fp_line (start -0.5 -0.4) (end -0.8 -0.1)
+      (stroke (width 0.1) (type solid)) (layer "F.Fab"))
+    (fp_line (start 0.8 -0.4) (end -0.5 -0.4)
+      (stroke (width 0.1) (type solid)) (layer "F.Fab"))
+    (fp_line (start 0.8 0.4) (end 0.8 -0.4)
+      (stroke (width 0.1) (type solid)) (layer "F.Fab"))
+    (pad "1" smd roundrect (at -0.7875 0 90) (size 0.875 0.95) (layers "F.Cu" "F.Paste" "F.Mask") (roundrect_rratio 0.25)
+      (net 2 "GND") (pinfunction "K") (pintype "passive"))
+    (pad "2" smd roundrect (at 0.7875 0 90) (size 0.875 0.95) (layers "F.Cu" "F.Paste" "F.Mask") (roundrect_rratio 0.25)
+      (net 46 "Net-(D3-A)") (pinfunction "A") (pintype "passive"))
+    (model "${KICAD6_3DMODEL_DIR}/Diode_SMD.3dshapes/D_0603_1608Metric.wrl"
       (offset (xyz 0 0 0))
       (scale (xyz 1 1 1))
@@
       (net 2 "GND") (pintype "passive"))
     (model "${KICAD6_3DMODEL_DIR}/Capacitor_SMD.3dshapes/C_0603_1608Metric.wrl"
+      (offset (xyz 0 0 0))
+      (scale (xyz 1 1 1))
+      (rotate (xyz 0 0 0))
+    )
+  )
+  (footprint "Resistor_SMD:R_0603_1608Metric" (layer "F.Cu")
+    (at 224.3 65.7)
+    (descr "Resistor SMD 0603 (1608 Metric), square (rectangular) end terminal, IPC_7351 nominal, (Body size source: IPC-SM-782 page 72, https://www.pcb-3d.com/wordpress/wp-content/uploads/ipc-sm-782a_amendment_1_and_2.pdf), generated with kicad-footprint-generator")
+    (tags "resistor")
+    (property "Manufacturer" "Generic")
+    (property "Part #" "Generic 0603 1K 1% Resistor")
+    (property "Sheetfile" "rocket2-trs.kicad_sch")
+    (property "Sheetname" "")
+    (property "ki_description" "Resistor, small US symbol")
+    (property "ki_keywords" "r resistor")
+    (attr smd)
+    (fp_text reference "R4" (at 0 -1.43) (layer "F.SilkS") hide
+        (effects (font (size 1 1) (thickness 0.15)))
+    )
+    (fp_text value "1K" (at 0 1.43) (layer "F.Fab")
+        (effects (font (size 1 1) (thickness 0.15)))
+    )
+    (fp_text user "${REFERENCE}" (at 0 0) (layer "F.Fab")
+        (effects (font (size 0.4 0.4) (thickness 0.06)))
+    )
+    (fp_line (start -0.237258 -0.5225) (end 0.237258 -0.5225)
+      (stroke (width 0.12) (type solid)) (layer "F.SilkS"))
+    (fp_line (start -0.237258 0.5225) (end 0.237258 0.5225)
+      (stroke (width 0.12) (type solid)) (layer "F.SilkS"))
+    (fp_line (start -1.48 -0.73) (end 1.48 -0.73)
+      (stroke (width 0.05) (type solid)) (layer "F.CrtYd"))
+    (fp_line (start -1.48 0.73) (end -1.48 -0.73)
+      (stroke (width 0.05) (type solid)) (layer "F.CrtYd"))
+    (fp_line (start 1.48 -0.73) (end 1.48 0.73)
+      (stroke (width 0.05) (type solid)) (layer "F.CrtYd"))
+    (fp_line (start 1.48 0.73) (end -1.48 0.73)
+      (stroke (width 0.05) (type solid)) (layer "F.CrtYd"))
+    (fp_line (start -0.8 -0.4125) (end 0.8 -0.4125)
+      (stroke (width 0.1) (type solid)) (layer "F.Fab"))
+    (fp_line (start -0.8 0.4125) (end -0.8 -0.4125)
+      (stroke (width 0.1) (type solid)) (layer "F.Fab"))
+    (fp_line (start 0.8 -0.4125) (end 0.8 0.4125)
+      (stroke (width 0.1) (type solid)) (layer "F.Fab"))
+    (fp_line (start 0.8 0.4125) (end -0.8 0.4125)
+      (stroke (width 0.1) (type solid)) (layer "F.Fab"))
+    (pad "1" smd roundrect (at -0.825 0) (size 0.8 0.95) (layers "F.Cu" "F.Paste" "F.Mask") (roundrect_rratio 0.25)
+      (net 49 "Net-(U1-PB8)") (pintype "passive"))
+    (pad "2" smd roundrect (at 0.825 0) (size 0.8 0.95) (layers "F.Cu" "F.Paste" "F.Mask") (roundrect_rratio 0.25)
+      (net 46 "Net-(D3-A)") (pintype "passive"))
+    (model "${KICAD6_3DMODEL_DIR}/Resistor_SMD.3dshapes/R_0603_1608Metric.wrl"
       (offset (xyz 0 0 0))
       (scale (xyz 1 1 1))
@@
   (via (at 199.7 108.3) (size 0.8) (drill 0.4) (layers "F.Cu" "B.Cu") (free) (net 2))
   (via (at 199.2 48.8) (size 0.8) (drill 0.4) (layers "F.Cu" "B.Cu") (free) (net 2))
+  (via (at 227.3 68.5) (size 0.8) (drill 0.4) (layers "F.Cu" "B.Cu") (free) (net 2))
   (via (at 218.6 72.6) (size 0.8) (drill 0.4) (layers "F.Cu" "B.Cu") (free) (net 2))
   (via (at 198.8 111.2) (size 0.8) (drill 0.4) (layers "F.Cu" "B.Cu") (free) (net 2))
@@
   (segment (start 217 97) (end 217 67.8) (width 0.25) (layer "B.Cu") (net 38))
   (segment (start 217 67.8) (end 213.9 64.7) (width 0.25) (layer "B.Cu") (net 38))
+  (segment (start 227.2875 65.7) (end 227.3 65.7125) (width 0.25) (layer "F.Cu") (net 46))
+  (segment (start 225.125 65.7) (end 227.2875 65.7) (width 0.25) (layer "F.Cu") (net 46))
+  (segment (start 220.1625 65.75) (end 223.425 65.75) (width 0.25) (layer "F.Cu") (net 49))
+  (segment (start 223.425 65.75) (end 223.475 65.7) (width 0.25) (layer "F.Cu") (net 49))
   (zone (net 2) (net_name "GND") (layers "F.Cu" "In1.Cu" "B.Cu") (hatch edge 0.5)
     (connect_pads thru_hole_only (clearance 0.2))

Commit message: TRS Update 1
Parts:
- moved J2 0.20 mm to (200.0, 44.8)
- moved R3 0.10 mm to (197.6, 108.4)
- moved R2 0.10 mm to (192.9, 108.4)
Routing:
- net GND: track 0.00 -> 296.9 mm
- net +3.3V: track 50.8 -> 210.2 mm, vias 13 -> 14
- removed copper zone on In2.Cu, net +3.3V
- removed copper zone on B.Cu, net GND
- removed copper zone on F.Cu, net GND
- removed copper zone on In1.Cu, net GND
Other:
- copper layers 4 -> 2

Commit message: TRS 1
Parts:
- TP15: value RADIO_DIO5 -> R_DIO5
- TP16: value RADIO_DIO4 -> R_DIO4
- TP17: value RADIO_DIO3 -> R_DIO3
- TP18: value RADIO_DIO2 -> R_DIO2
- TP19: value RADIO_DIO1 -> R_DIO1
- TP20: value RADIO_DIO0 -> R_DIO0
- TP4: value RADIO_nRST -> R_nRST
- TP5: value RADIO_nCS -> R_nCS
- TP6: value RADIO_SCK -> R_SCK
- TP7: value RADIO_MOSI -> R_MOSI
- TP8: value RADIO_MISO -> R_MISO
- moved TP17 19.0 mm to (177.0, 51.6)
- moved TP5 18.9 mm to (178.8, 61.8), turned to 90 degrees
- moved TP4 18.6 mm to (181.2, 61.8), turned to 90 degrees
- moved TP15 18.2 mm to (183.6, 61.8), turned to 90 degrees
- moved TP16 14.9 mm to (179.4, 54.0)
- moved TP7 11.0 mm to (183.6, 64.0)
- moved TP6 9.39 mm to (183.6, 68.8)
- moved TP8 7.93 mm to (183.6, 66.4)
- moved TP20 6.84 mm to (183.4, 49.2), turned to 90 degrees
- moved TP19 4.54 mm to (183.5, 51.6)
- moved TP18 3.91 mm to (183.5, 54.0)
- moved J2 0.20 mm to (200.0, 45.0)
- moved R3 0.10 mm to (197.6, 108.3)
- moved R2 0.10 mm to (192.9, 108.3)
Routing:
- net GND: track 296.9 -> 15.6 mm
- net RADIO_DIO5: track 26.2 -> 77.8 mm, vias 2 -> 3
- net RADIO_nRST: track 23.7 -> 67.1 mm, vias 0 -> 2
- net RADIO_nCS: track 27.7 -> 55.4 mm, vias 0 -> 2
- net RADIO_DIO3: track 30.3 -> 56.1 mm
- net RADIO_DIO4: track 32.9 -> 55.8 mm
- net RADIO_SCK: track 30.3 -> 42.9 mm, vias 0 -> 2
- net RADIO_MOSI: track 34.8 -> 43.7 mm
- net RADIO_DIO0: track 39.3 -> 47.5 mm
- net +3.3V: track 210.2 -> 203.8 mm, vias 14 -> 7
- net RADIO_MISO: track 35.4 -> 41.3 mm
- net RADIO_DIO1: track 39.6 -> 43.3 mm
- net RADIO_DIO2: track 39.6 -> 39.1 mm
- added copper zone on B.Cu, net GND
- added copper zone on F.Cu, net GND
Other:
- board size 50 x 80 mm -> 57 x 80 mm
