File: rocket2-trs-hardware.kicad_sch (KiCad schematic)
At the start: 63 parts, among them J1 Conn_01x02_Pin, J2 USB_C_Receptacle_USB2.0_16P, J3 ARM Cortex Debug, J4 Conn_Coaxial, J5 Screw_Terminal_01x02, J7 Screw_Terminal_01x02, Q1 Q_PMOS, Q2 NMOS, Q3 NMOS, U1 AP63205WU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

Commit message: TRS production ready
Parts:
- added C17: 0.1uf, Capacitor_SMD:C_0603_1608Metric_Pad1.08x0.95mm_HandSolder, symbol Device:C
- added R6, R8: 1.5k, Resistor_SMD:R_0603_1608Metric_Pad0.98x0.95mm_HandSolder, symbol Device:R
- U7: value opto -> TLP3553A(TP1,F
- U8: value opto -> TLP3553A(TP1,F; Part# (none) -> TLP3553A(TP1,F
Connections:
- net GND: now also C17.2, R6.2, R8.2
- net NRST_LORA: now reaches U2.11 (PA1)
- net NRST_LORA: now also U6.5 (RST)
- net NRST: now reaches U2.7 (NRST)
- net NRST: now also J3.10 (~{RST}), C17.1
- net at J2.A5 (CC1): now also R8.1
- net at J2.B5 (CC2): now also R6.1
- no-connect marks 8 -> 6
Other:
- moved on the sheet: U6
